File: I2C-Keypad-Backpack.brd (EAGLE design)
At the start: 30.5 x 26.7 mm, 18 parts, among them U1 MCP23008

Commit message: Rev C
Other:
- board text added: "I2C Keypad BKPK (C)"
- board text added: "dcity.org"
Changed lines of the file:
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@@
 <?xml version="1.0" encoding="utf-8"?>
 <!DOCTYPE eagle SYSTEM "eagle.dtd">
-<eagle version="7.5.0">
+<eagle version="9.1.3">
 <drawing>
 <settings>
 <setting alwaysvectorfont="no"/>
+<setting keepoldvectorfont="yes"/>
 <setting verticaltext="up"/>
 </settings>
@@
 <text x="22.733" y="6.604" size="0.889" layer="21" font="vector" ratio="15" rot="R90">A1</text>
 <text x="25.273" y="6.477" size="0.889" layer="21" font="vector" ratio="15" rot="SR90">A2</text>
-<text x="27.051" y="10.541" size="0.889" layer="21" font="vector" ratio="15" rot="R180">I2C Keypad BKPK (B)</text>
+<text x="27.051" y="10.541" size="0.889" layer="21" font="vector" ratio="15" rot="R180">I2C Keypad BKPK (C)</text>
 <text x="7.112" y="24.638" size="0.889" layer="22" font="vector" ratio="15" rot="MR270">I2C Keypad BKPK (B)</text>
 <text x="16.764" y="9.017" size="0.889" layer="21" font="vector" ratio="15" rot="R270">SCL</text>
@@
 <rectangle x1="22.987" y1="1.016" x2="24.13" y2="2.794" layer="43"/>
 <text x="25.527" y="18.923" size="1.524" layer="21" font="vector" ratio="10" rot="R270">wht.io</text>
-<text x="5.461" y="19.939" size="1.524" layer="22" font="vector" ratio="10" rot="MR270">wht.io</text>
+<text x="5.461" y="21.209" size="1.524" layer="22" font="vector" ratio="10" rot="MR270">dcity.org</text>
 <rectangle x1="12.5095" y1="1.3335" x2="14.1605" y2="2.3495" layer="43" rot="R90"/>
 <rectangle x1="18.034" y1="19.304" x2="19.685" y2="20.701" layer="43"/>
@@
 <param name="dpMaxLengthDifference" value="10mm"/>
 <param name="dpGapFactor" value="2.5"/>
-<param name="checkGrid" value="0"/>
 <param name="checkAngle" value="1"/>
 <param name="checkFont" value="1"/>
 <param name="checkRestrict" value="1"/>
+<param name="checkStop" value="0"/>
+<param name="checkValues" value="0"/>
+<param name="checkNames" value="1"/>
+<param name="checkWireStubs" value="1"/>
+<param name="checkPolygonWidth" value="0"/>
 <param name="useDiameter" value="13"/>
 <param name="maxErrors" value="50"/>
@@
 <element name="LOGO1" library="0" package="OSHW-LOGO-S" value="OSHW-LOGOS" x="28.067" y="1.651"/>
 <element name="J3" library="0" package="1X08_LOCK" value="" x="29.21" y="5.08" smashed="yes" rot="R90">
-<attribute name="NAME" x="29.7942" y="2.8702" size="0.889" layer="25" font="vector" ratio="15" rot="R180"/>
+<attribute name="NAME" x="29.7942" y="25.7302" size="0.889" layer="25" font="vector" ratio="15" rot="R180"/>
 <attribute name="VALUE" x="32.385" y="3.81" size="1.27" layer="27" rot="R90"/>
 </element>
@@
 </signal>
 </signals>
+<mfgpreviewcolors>
+<mfgpreviewcolor name="soldermaskcolor" color="0xC8008000"/>
+<mfgpreviewcolor name="silkscreencolor" color="0xFFFEFEFE"/>
+<mfgpreviewcolor name="backgroundcolor" color="0xFF282828"/>
+<mfgpreviewcolor name="coppercolor" color="0xFFFFBF00"/>
+<mfgpreviewcolor name="substratecolor" color="0xFF786E46"/>
+</mfgpreviewcolors>
 </board>
 </drawing>

Commit message: Rev D
Parts:
- J1, J2: value (none) -> QWIIC_RIGHT_ANGLE; device 0:HW4-SMD-2.0-90D -> 0:JST04_1MM_RA
- moved LOGO1 34.4 mm to (2.29, 24.4)
- moved J1 12.9 mm to (4.95, 18.2), turned to 270 degrees
- moved J2 12.9 mm to (4.95, 8.51), turned to 270 degrees
- moved J3 6.35 mm to (22.9, 5.08)
- moved J4 6.35 mm to (18.4, 24.1)
- moved R2 6.35 mm to (15.9, 1.91)
- moved R3 6.35 mm to (18.4, 1.91)
- moved SJ2 6.35 mm to (15.9, 5.08)
- moved SJ3 6.35 mm to (18.4, 5.08)
- moved C1 6.35 mm to (8.26, 23.5)
- moved C2 6.35 mm to (10.8, 23.5)
- moved R4 6.35 mm to (8.26, 1.91)
- moved R5 6.35 mm to (10.8, 1.91)
- moved SJ4 6.35 mm to (8.26, 5.08)
- moved SJ5 6.35 mm to (10.8, 5.08)
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Connections:
- net GND: now also J1.1, J2.1; no longer J1.4, J2.4
- net SCL: now also J1.4, J2.4; no longer J1.1, J2.1
- net SDA: now also J1.3, J2.3; no longer J1.2, J2.2
- net VCC: now also J1.2, J2.2; no longer J1.3, J2.3
Routing:
- net SCL: track 57.3 -> 53.2 mm
- net VCC: track 71.5 -> 68.0 mm
- net SDA: track 27.8 -> 24.4 mm
Other:
- board size 30.5 x 26.7 mm -> 24.1 x 26.7 mm
- board text added: "GND"
- board text added: "I2C Keypad BKPK (D)"
- board text added: "VCC"
- board text removed: "I2C Keypad BKPK (B)"
- board text removed: "I2C Keypad BKPK (C)"
- board text removed: "wht.io"
