File: I2C-Keypad-Backpack.sch (EAGLE design)
At the start: 18 parts, among them U1 MCP23008

Commit message: Rev D
Parts:
- J1, J2: value (none) -> QWIIC_RIGHT_ANGLE; device 0:GROVE-CONNECTOR-SMD-90D(4+2P-2.0) -> 0:QWIIC_CONNECTORJS-1MM
Connections:
- net GND: now also J1.1, J2.1; no longer J1.4, J2.4
- net SCL: now also J1.4, J2.4; no longer J1.1, J2.1
- net SDA: now also J1.3, J2.3; no longer J1.2, J2.2
- net VCC: now also J1.2, J2.2; no longer J1.3, J2.3
